Commit message: commit current save

File: eufs/install/eufs_sensors/share/eufs_sensors/urdf/VLP-16R.urdf.xacro (robot description, xacro)
@@ -1 +1,100 @@
-/home/andrewwhong/classes/16833/iSAM2_SLAM/eufs/eufs_sim/eufs_sensors/urdf/VLP-16R.urdf.xacro
+<?xml version="1.0"?>
+<robot xmlns:xacro="http://www.ros.org/wiki/xacro" name="VLP-16">
+  <xacro:property name="M_PI" value="3.1415926535897931" />
+  <xacro:macro name="VLP-16R" params="*origin parent:=base_footprint name:=velodyne active topic:=/velodyne_points hz:=10 lasers:=40 samples:=350 min_range:=0.2 max_range:=100.0 noise:=0.008 min_angle:=-2 max_angle:=2">
+    <joint name="${name}_base_mount_joint" type="fixed">
+      <xacro:insert_block name="origin" />
+      <parent link="${parent}"/>
+      <child link="${name}_base_link"/>
+    </joint>
+    <link name="${name}_base_link">
+      <inertial>
+        <mass value="0.83"/>
+        <origin xyz="0 0 0.03585"/>
+        <inertia ixx="${(0.83 * (3.0*0.0516*0.0516 + 0.0717*0.0717)) / 12.0}" ixy="0" ixz="0"
+          iyy="${(0.83 * (3.0*0.0516*0.0516 + 0.0717*0.0717)) / 12.0}" iyz="0"
+          izz="${0.5 * 0.83 * (0.0516*0.0516)}"/>
+      </inertial>
+      <visual>
+        <geometry>
+          <mesh filename="file://$(find eufs_sensors)/meshes/VLP16_base_1.dae" />
+        </geometry>
+      </visual>
+      <visual>
+        <geometry>
+          <mesh filename="file://$(find eufs_sensors)/meshes/VLP16_base_2.dae" />
+        </geometry>
+      </visual>
+      <collision>
+        <origin rpy="0 0 0" xyz="0 0 0.03585"/>
+        <geometry>
+          <cylinder radius="0.0516" length="0.0717"/>
+        </geometry>
+      </collision>
+    </link>
+    <joint name="${name}_base_scan_joint" type="fixed" >
+      <origin xyz="0 0 0.0377" rpy="0 0 0" />
+      <parent link="${name}_base_link" />
+      <child link="${name}"/>
+    </joint>
+    <link name="${name}">
+      <inertial>
+        <mass value="0.01"/>
+        <origin xyz="0 0 0"/>
+        <inertia ixx="1e-7" ixy="0" ixz="0" iyy="1e-7" iyz="0" izz="1e-7"/>
+      </inertial>
+      <visual>
+        <origin xyz="0 0 -0.0377" />
+        <geometry>
+          <mesh filename="file://$(find eufs_sensors)/meshes/VLP16_scan.dae" />
+        </geometry>
+      </visual>
+    </link>
+    <!-- Simulate raw perception sensors only if we're not using the abstracted perception simulation -->
+    <xacro:unless value="${active}">
+      <!-- Gazebo requires the velodyne_gazebo_plugins package -->
+      <gazebo reference="${name}">
+        <sensor type="ray" name="${name}-VLP16">
+          <always_on>true</always_on>
+          <pose>0 0 0 0 0 0</pose>
+          <visualize>false</visualize>
+          <update_rate>${hz}</update_rate>
+          <ray>
+            <scan>
+              <horizontal>
+                <samples>${samples}</samples>
+                <resolution>1.0</resolution>
+                <min_angle>${min_angle}</min_angle>
+                <max_angle>${max_angle}</max_angle>
+              </horizontal>
+              <vertical>
+                <samples>${lasers}</samples>
+                <resolution>1.0</resolution>
+                <min_angle>-${15.0*M_PI/180.0}</min_angle>
+                <max_angle> ${15.0*M_PI/180.0}</max_angle>
+              </vertical>
+            </scan>
+            <range>
+              <min>${min_range}</min>
+              <max>${max_range}</max>
+              <resolution>0.001</resolution>
+            </range>
+            <noise>
+              <type>gaussian</type>
+              <mean>0.0</mean>
+              <stddev>${noise}</stddev>
+            </noise>
+          </ray>
+          <plugin name="gazebo_ros_laser_controller" filename="libgazebo_ros_ray_sensor.so">
+            <ros>
+              <remapping>~/out:=${topic}</remapping>
+            </ros>
+            <frame_name>${name}</frame_name>
+            <radiation_type>infrared</radiation_type>
+            <output_type>sensor_msgs/PointCloud2</output_type>
+          </plugin>
+        </sensor>
+      </gazebo>
+    </xacro:unless>
+  </xacro:macro>
+</robot>

File: eufs/install/eufs_sensors/share/eufs_sensors/urdf/all_sensors.urdf.xacro (robot description, xacro)
@@ -1 +1,14 @@
-/home/andrewwhong/classes/16833/iSAM2_SLAM/eufs/eufs_sim/eufs_sensors/urdf/all_sensors.urdf.xacro
+<?xml version="1.0"?>
+<robot name="all_sensors" xmlns:xacro="http://www.ros.org/wiki/xacro">
+  <!-- This file unifies all sensors that can be used on simulation, defined as xacro:macros -->
+  <!-- GPS -->
+  <xacro:include filename="$(find eufs_sensors)/urdf/gps.urdf.xacro"/>
+  <!-- Velodyne VLP-16R -->
+  <xacro:include filename="$(find eufs_sensors)/urdf/VLP-16R.urdf.xacro"/>
+  <!-- Magnetometer-->
+  <xacro:include filename="$(find eufs_sensors)/urdf/magnetometer.urdf.xacro"/>
+  <!--IMU -->
+  <xacro:include filename="$(find eufs_sensors)/urdf/imu.urdf.xacro"/>
+  <!-- ZED Stereo camera -->
+  <xacro:include filename="$(find eufs_sensors)/urdf/zed.urdf.xacro"/>
+</robot>

File: eufs/install/eufs_sensors/share/eufs_sensors/urdf/gps.urdf.xacro (robot description, xacro)
@@ -1 +1,92 @@
-/home/andrewwhong/classes/16833/iSAM2_SLAM/eufs/eufs_sim/eufs_sensors/urdf/gps.urdf.xacro
+<?xml version="1.0"?>
+<robot name="sensor_gps" xmlns:xacro="http://www.ros.org/wiki/xacro">
+    <xacro:macro name="sensor_gps" params="prefix parent *origin">
+        <!-- ANTENNA GPS -->
+        <joint name="${prefix}_joint" type="fixed">
+            <axis xyz="0 1 0"/>
+            <xacro:insert_block name="origin"/>
+            <parent link="${parent}"/>
+            <child link="${prefix}_base_link"/>
+        </joint>
+        <link name="${prefix}_base_link">
+            <inertial>
+                <mass value="0.001"/>
+                <origin rpy="0 0 0" xyz="0 0 0"/>
+                <inertia ixx="0.0001" ixy="0" ixz="0" iyy="0.000001" iyz="0" izz="0.0001"/>
+            </inertial>
+            <visual>
+                <origin rpy="0 0 0" xyz="0 0 0"/>
+                <geometry>
+                    <box size="0.001 0.001 0.001"/>
+                </geometry>
+            </visual>
+            <collision>
+                <origin rpy="0 0 0" xyz="0 0 0"/>
+                <geometry>
+                    <box size=".001 .001 .001"/>
+                </geometry>
+            </collision>
+<!--        <visual>-->
+<!--            <origin rpy="0 0 0" xyz="0 0 0"/>-->
+<!--            <material name="gps_color">-->
+<!--                <color rgba="1 1 1 1"/>-->
+<!--            </material>-->
+<!--            <geometry>-->
+<!--                <mesh filename="file://$(find eufs_sensors)/meshes/antenna_3GO16.stl" scale="1.0 1.0 1.0"/>-->
+<!--            </geometry>-->
+<!--        </visual>-->
+<!--        <collision>-->
+<!--            <origin rpy="0 0 0" xyz="0 0 0"/>-->
+<!--            <geometry>-->
+<!--                <mesh filename="file://$(find eufs_sensors)/meshes/antenna_3GO16.stl" scale="1.0 1.0 1.0"/>-->
+<!--            </geometry>-->
+<!--        </collision>-->
+        </link>
+        <gazebo reference="${prefix}_base_link">
+            <material>Gazebo/White</material>
+            <gravity>true</gravity>
+        </gazebo>
+        <gazebo reference="${prefix}_base_link">
+            <sensor name="gps" type="gps">
+                <always_on>true</always_on>
+                <update_rate>5</update_rate>
+                <gps>
+                    <position_sensing>
+                        <horizontal>
+                            <noise type="gaussian">
+                                <mean>0.0</mean>
+                                <stddev>2</stddev>
+                            </noise>
+                        </horizontal>
+                        <vertical>
+                            <noise type="gaussian">
+                                <mean>0.0</mean>
+                                <stddev>2.5</stddev>
+                            </noise>
+                        </vertical>
+                    </position_sensing>
+                    <velocity_sensing>
+                        <horizontal>
+                            <noise type="gaussian">
+                                <mean>0.0</mean>
+                                <stddev>0.1</stddev>
+                            </noise>
+                        </horizontal>
+                        <vertical>
+                            <noise type="gaussian">
+                                <mean>0.0</mean>
+                                <stddev>0.1</stddev>
+                            </noise>
+                        </vertical>
+                    </velocity_sensing>
+                </gps>
+                <plugin name="${prefix}_controller" filename="libgazebo_ros_gps_sensor.so">
+                    <ros>
+                        <remapping>~/out:=${prefix}</remapping>
+                    </ros>
+                    <frame_name>${prefix}_base_link</frame_name>
+                </plugin>
+            </sensor>
+        </gazebo>
+    </xacro:macro>
+</robot>

File: eufs/install/eufs_sensors/share/eufs_sensors/urdf/imu.urdf.xacro (robot description, xacro)
@@ -1 +1,89 @@
-/home/andrewwhong/classes/16833/iSAM2_SLAM/eufs/eufs_sim/eufs_sensors/urdf/imu.urdf.xacro
+<?xml version="1.0"?>
+<robot name="sensor_imu" xmlns:xacro="http://www.ros.org/wiki/xacro">
+    <xacro:macro name="sensor_imu" params="prefix parent topic_prefix *origin noise:=0.08">
+        <joint name="${prefix}_base_joint" type="fixed">
+            <axis xyz="1 0 0"/>
+            <xacro:insert_block name="origin"/>
+            <parent link="${parent}"/>
+            <child link="${prefix}_base_link"/>
+        </joint>
+        <link name="${prefix}_base_link">
+            <inertial>
+                <mass value="0.001"/>
+                <origin rpy="0 0 0" xyz="0 0 0"/>
+                <inertia ixx="0.0001" ixy="0" ixz="0" iyy="0.000001" iyz="0" izz="0.0001"/>
+            </inertial>
+            <visual>
+                <origin rpy="0 0 0" xyz="0 0 0"/>
+                <geometry>
+                    <box size="0.001 0.001 0.001"/>
+                </geometry>
+            </visual>
+            <collision>
+                <origin rpy="0 0 0" xyz="0 0 0"/>
+                <geometry>
+                    <box size=".001 .001 .001"/>
+                </geometry>
+            </collision>
+        </link>
+        <gazebo reference="${prefix}_base_link">
+            <gravity>true</gravity>
+            <sensor name="{prefix}_sensor" type="imu">
+                <always_on>true</always_on>
+                <update_rate>1000</update_rate>
+                <visualize>true</visualize>
+                <topic>imu/data</topic>
+                <imu>
+                    <angular_velocity>
+                        <x>
+                            <noise type="gaussian">
+                                <mean>0.0</mean>
+                                <stddev>${noise}</stddev>
+                            </noise>
+                        </x>
+                        <y>
+                            <noise type="gaussian">
+                                <mean>0.0</mean>
+                                <stddev>${noise}</stddev>
+                            </noise>
+                        </y>
+                        <z>
+                            <noise type="gaussian">
+                                <mean>0.0</mean>
+                                <stddev>${noise}</stddev>
+                            </noise>
+                        </z>
+                    </angular_velocity>
+                    <linear_acceleration>
+                        <x>
+                            <noise type="gaussian">
+                                <mean>0.0</mean>
+                                <stddev>${noise}</stddev>
+                            </noise>
+                        </x>
+                        <y>
+                            <noise type="gaussian">
+                                <mean>0.0</mean>
+                                <stddev>${noise}</stddev>
+                            </noise>
+                        </y>
+                        <z>
+                            <noise type="gaussian">
+                                <mean>0.0</mean>
+                                <stddev>${noise}</stddev>
+                            </noise>
+                        </z>
+                    </linear_acceleration>
+                </imu>
+                <plugin filename="libgazebo_ros_imu_sensor.so" name="${prefix}">
+                    <ros>
+                        <remapping>~/out:=${topic_prefix}/imu/data</remapping>
+                    </ros>
+                    <frame_name>${prefix}_base_link</frame_name>
+                    <initial_orientation_as_reference>false</initial_orientation_as_reference>
+                </plugin>
+                <pose>0 0 0 0 0 0</pose>
+            </sensor>
+        </gazebo>
+    </xacro:macro>
+</robot>

File: eufs/install/eufs_sensors/share/eufs_sensors/urdf/magnetometer.urdf.xacro (robot description, xacro)
@@ -1 +1,36 @@
-/home/andrewwhong/classes/16833/iSAM2_SLAM/eufs/eufs_sim/eufs_sensors/urdf/magnetometer.urdf.xacro
+<?xml version="1.0"?>
+<robot name="sensor_magnetometer" xmlns:xacro="http://www.ros.org/wiki/xacro">
+    <xacro:macro name="sensor_magnetometer" params="prefix parent *origin noise:=0.08">
+        <joint name="${prefix}_base_joint" type="fixed">
+            <axis xyz="1 0 0"/>
+            <xacro:insert_block name="origin"/>
+            <parent link="${parent}"/>
+            <child link="${prefix}_base_link"/>
+        </joint>
+        <link name="${prefix}_base_link">
+            <inertial>
+                <mass value="0.001"/>
+                <origin rpy="0 0 0" xyz="0 0 0"/>
+                <inertia ixx="0.0001" ixy="0" ixz="0" iyy="0.000001" iyz="0" izz="0.0001"/>
+            </inertial>
+            <visual>
+                <origin rpy="0 0 0" xyz="0 0 0"/>
+                <geometry>
+                    <box size="0.001 0.001 0.001"/>
+                </geometry>
+            </visual>
+            <collision>
+                <origin rpy="0 0 0" xyz="0 0 0"/>
+                <geometry>
+                    <box size=".001 .001 .001"/>
+                </geometry>
+            </collision>
+        </link>
+        <gazebo>
+            <plugin filename="libhector_gazebo_ros_magnetic.so" name="${prefix}">
+                <robotNamespace> ${prefix} </robotNamespace>
+                <topicName> sbg/magnetic </topicName>
+            </plugin>
+        </gazebo>
+    </xacro:macro>
+</robot>

File: eufs/install/eufs_sensors/share/eufs_sensors/urdf/zed.urdf.xacro (robot description, xacro)
@@ -1 +1,145 @@
-/home/andrewwhong/classes/16833/iSAM2_SLAM/eufs/eufs_sim/eufs_sensors/urdf/zed.urdf.xacro
+<?xml version="1.0"?>
+<robot name="zed_camera"
+  xmlns:xacro="http://www.ros.org/wiki/xacro">
+  <xacro:macro name="zed_camera" params="prefix parent *origin active">
+    <joint name="${prefix}_base_joint" type="fixed">
+      <axis xyz="1 0 0"/>
+      <xacro:insert_block name="origin"/>
+      <parent link="${parent}"/>
+      <child link="${prefix}_camera_center"/>
+    </joint>
+    <link name="${prefix}_camera_center">
+      <visual>
+        <origin xyz="0 0 0" rpy="0 0 0"/>
+        <geometry>
+          <mesh filename="file://$(find eufs_sensors)/meshes/zed.dae" />
+        </geometry>
+        <material name="light_grey">
+          <color rgba="0.8 0.8 0.8 0.8"/>
+        </material>
+      </visual>
+    </link>
+    <!-- Left and right frames -->
+    <link name="${prefix}_left_camera_frame"/>
+    <link name="${prefix}_right_camera_frame"/>
+    <link name="${prefix}_left_camera_optical_frame"/>
+    <link name="${prefix}_right_camera_optical_frame"/>
+    <joint name="${prefix}_left_camera_joint" type="fixed">
+      <parent link="${prefix}_camera_center"/>
+      <child link="${prefix}_left_camera_frame"/>
+      <origin xyz="0 0.06 0" rpy="0 0 0" />
+    </joint>
+    <joint name="${prefix}_right_camera_joint" type="fixed">
+      <parent link="${prefix}_camera_center"/>
+      <child link="${prefix}_right_camera_frame"/>
+      <origin xyz="0 -0.06 0" rpy="0 0 0" />
+    </joint>
+    <joint name="left_camera_optical_joint" type="fixed">
+      <origin xyz="0 0 0" rpy="0.0 0.0 0.0" />
+      <parent link="${prefix}_left_camera_frame" />
+      <child link="${prefix}_left_camera_optical_frame"/>
+    </joint>
+    <joint name="right_camera_optical_joint" type="fixed">
+      <origin xyz="0 0 0" rpy="0.0 0.0 0.0" />
+      <parent link="${prefix}_right_camera_frame" />
+      <child link="${prefix}_right_camera_optical_frame"/>
+    </joint>
+    <!-- depth frame -->
+    <link name="${prefix}_depth_camera_frame"/>
+    <joint name="${prefix}_depth_camera" type="fixed">
+      <parent link="${prefix}_camera_center"/>
+      <child link="${prefix}_depth_camera_frame"/>
+      <origin xyz="0 0.06 0" rpy="0 0 0" />
+    </joint>
+    <!-- Simulate raw perception sensors only if we're not using the abstracted perception simulation -->
+    <xacro:unless value="${active}">
+      <gazebo reference="${prefix}_left_camera_optical_frame">
+        <sensor type="multicamera" name="stereo_camera">
+          <!-- see MultiSenseSLPlugin.h for available modes -->
+          <always_on>true</always_on>
+          <update_rate>60.0</update_rate>
+          <visualize>true</visualize>
+          <camera name="${prefix}_left">
+            <pose>0 0.0 0 0 0 0</pose>
+            <horizontal_fov>1.91986</horizontal_fov>
+            <image>
+              <width>1280</width>
+              <height>720</height>
+              <format>B8G8R8</format>
+            </image>
+            <clip>
+              <near>0.5</near>
+              <far>20</far>
+            </clip>
+            <noise>
+              <type>gaussian</type>
+              <mean>0.0</mean>
+              <stddev>0.007</stddev>
+            </noise>
+          </camera>
+          <camera name="${prefix}_right">
+            <pose>0 -0.12 0 0 0 0</pose>
+            <horizontal_fov>1.91986</horizontal_fov>
+            <image>
+              <width>1280</width>
+              <height>720</height>
+              <format>B8G8R8</format>
+            </image>
+            <clip>
+              <near>0.5</near>
+              <far>20</far>
+            </clip>
+            <noise>
+              <type>gaussian</type>
+              <mean>0.0</mean>
+              <stddev>0.007</stddev>
+            </noise>
+          </camera>
+          <plugin name="stereo_camera_controller" filename="libgazebo_ros_camera.so">
+            <ros>
+              <parameter name="update_rate" type="double">60.0</parameter>
+              <remapping>/zed/zed_left/camera_info:=/zed/left/camera_info</remapping>
+              <remapping>/zed/zed_left/image_raw:=/zed/left/image_rect_color</remapping>
+              <remapping>/zed/zed_right/camera_info:=/zed/right/camera_info</remapping>
+              <remapping>/zed/zed_right/image_raw:=/zed/right/image_rect_color</remapping>
+            </ros>
+            <camera_name>${prefix}</camera_name>
+            <frame_name>${prefix}_left_camera_optical_frame</frame_name>
+            <hack_baseline>0.120</hack_baseline>
+            <triggered>false</triggered>
+          </plugin>
+        </sensor>
+        <!-- Depth simulation -->
+        <sensor name="stereo_depth" type="depth">
+          <always_on>true</always_on>
+          <update_rate>60.0</update_rate>
+          <visualize>false</visualize>
+          <camera>
+            <horizontal_fov>1.91986</horizontal_fov>
+            <image>
+              <width>1280</width>
+              <height>720</height>
+              <format>B8G8R8</format>
+            </image>
+            <depth_camera>
+            </depth_camera>
+            <clip>
+              <near>0.5</near>
+              <far>20.0</far>
+            </clip>
+          </camera>
+          <plugin name="${prefix}_controller" filename="libgazebo_ros_camera.so">
+            <ros>
+              <parameter name="update_rate" type="double">60.0</parameter>
+            </ros>
+            <camera_name>${prefix}</camera_name>
+            <frame_name>${prefix}_depth_camera_frame</frame_name>
+            <hack_baseline>0.120</hack_baseline>
+            <max_depth>20.0</max_depth>
+            <min_depth>0.5</min_depth>
+          </plugin>
+        </sensor>
+      </gazebo>
+    </xacro:unless>
+  </xacro:macro>
+</robot>
